File: kicad/k1-aioc/k1-aioc.kicad_pcb (KiCad board)
At the start: 2 copper layers, 21 x 31.5 mm, 50 parts, among them J1 USB4105-GF-A, J2 Conn_01x07_Male, Q1 BC847BS, U1 MIC5330-SSYML, U2 STM32F373CBTx, Y1 8MHz/20pF

Commit message: kicad update
Parts:
- Q1: value BC847BS -> MMDT3904
- U1: value MIC5330-SSYML -> MIC5332-SSYMT
Changed lines of the file:
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@@
       (effects (font (size 0.5 0.5) (thickness 0.1)))
     )
-    (fp_text value "BC847BS" (at 0 2) (layer "F.Fab") hide
+    (fp_text value "MMDT3904" (at 0 2) (layer "F.Fab") hide
       (effects (font (size 1 1) (thickness 0.15)))
     )
@@
       (effects (font (size 1 1) (thickness 0.15)))
     )
-    (fp_text value "MIC5330-SSYML" (at 0 1.95 -90) (layer "F.Fab") hide
+    (fp_text value "MIC5332-SSYMT" (at 0 1.95 -90) (layer "F.Fab") hide
       (effects (font (size 1 1) (thickness 0.15)))
     )
@@
       (net 1 "GND") (pinfunction "GND") (pintype "power_in"))
     (pad "3" smd roundrect (at -0.975 0.25 270) (size 0.75 0.25) (layers "F.Cu" "F.Paste" "F.Mask") (roundrect_rratio 0.25)
-      (net 22 "Net-(C3-Pad1)") (pinfunction "BYP") (pintype "passive"))
+      (net 22 "Net-(C3-Pad1)") (pinfunction "POR2") (pintype "open_collector"))
     (pad "4" smd roundrect (at -0.975 0.75 270) (size 0.75 0.25) (layers "F.Cu" "F.Paste" "F.Mask") (roundrect_rratio 0.25)
       (net 27 "/VIN") (pinfunction "EN2") (pintype "input"))
