File: kicad/k1-aioc/k1-aioc.kicad_sch (KiCad schematic)
At the start: 49 parts, among them J1 USB4105-GF-A, J2 Conn_01x07_Male, Q1 BC847BS, U1 MIC5330-SSYML, U2 STM32F373CBTx, Y1 8MHz/20pF

Commit message: kicad update
Parts:
- D1: LCSC C72043 -> C2986059
- Q1: value BC847BS -> MMDT3904; LCSC C8653 -> C83572
- U1: value MIC5330-SSYML -> MIC5332-SSYMT; symbol aioc:MIC5330-SSYML -> aioc:MIC5332-SSYMT; LCSC C144168 -> C153276
Other:
- note added: "U1: MIC5332-SSYMT (LCSC C153276) is a drop-in for the unobtainable MIC5330-SSYML. Pin 3 = POR2 (open-drain reset output, unused; C3 is harmless). Pin 6 = CSET2: leave OPEN, never connect to GND."
Changed lines of the file:
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@@
       (effects (font (size 1.27 1.27)) (justify left))
     )
-    (property "Value" "BC847BS" (id 1) (at 219.71 69.8499 0)
+    (property "Value" "MMDT3904" (id 1) (at 219.71 69.8499 0)
       (effects (font (size 1.27 1.27)) (justify left))
     )
@@
       (effects (font (size 1.27 1.27)) hide)
     )
-    (property "LCSC" "C8653" (id 4) (at 219.71 67.3099 0)
+    (property "LCSC" "C83572" (id 4) (at 219.71 67.3099 0)
       (effects (font (size 1.27 1.27)) hide)
     )
@@
       (effects (font (size 1.27 1.27)) hide)
     )
-    (property "LCSC" "C72043" (id 4) (at 157.1625 156.21 0)
+    (property "LCSC" "C2986059" (id 4) (at 157.1625 156.21 0)
       (effects (font (size 1.27 1.27)) hide)
     )
@@
       (effects (font (size 1.27 1.27)) (justify left))
     )
-    (property "Value" "BC847BS" (id 1) (at 219.71 45.7199 0)
+    (property "Value" "MMDT3904" (id 1) (at 219.71 45.7199 0)
       (effects (font (size 1.27 1.27)) (justify left))
     )
@@
       (effects (font (size 1.27 1.27)) hide)
     )
-    (property "LCSC" "C8653" (id 4) (at 219.71 43.1799 0)
+    (property "LCSC" "C83572" (id 4) (at 219.71 43.1799 0)
       (effects (font (size 1.27 1.27)) hide)
     )
@@
     (pin "1")
   )
-  (symbol (lib_id "aioc:MIC5330-SSYML") (at 106.68 35.56 0) (unit 1)
+  (text "U1: MIC5332-SSYMT (LCSC C153276) is a drop-in for the unobtainable MIC5330-SSYML.\nPin 3 = POR2 (open-drain reset output, unused; C3 is harmless).\nPin 6 = CSET2: leave OPEN, never connect to GND."
+    (at 88.9 60.96 0)
+    (effects (font (size 1.27 1.27)) (justify left bottom))
+  )
+  (symbol (lib_id "aioc:MIC5332-SSYMT") (at 106.68 35.56 0) (unit 1)
     (in_bom yes) (on_board yes) (fields_autoplaced)
     (property "Reference" "U1" (id 0) (at 106.68 25.4 0))
-    (property "Value" "MIC5330-SSYML" (id 1) (at 106.68 27.94 0))
+    (property "Value" "MIC5332-SSYMT" (id 1) (at 106.68 27.94 0))
     (property "Footprint" "AIOC:Micrel_MLF-8-1EP_2x2mm_P0.5mm_EP0.6x1.2mm" (id 2) (at 144.78 41.91 0)
       (effects (font (size 1.27 1.27)) hide)
     )
-    (property "Datasheet" "http://ww1.microchip.com/downloads/en/DeviceDoc/mic5330.pdf" (id 3) (at 106.68 26.67 0)
-      (effects (font (size 1.27 1.27)) hide)
-    )
-    (property "LCSC" "C144168" (id 4) (at 106.68 35.56 0)
+    (property "Datasheet" "https://ww1.microchip.com/downloads/aemDocuments/documents/APID/ProductDocuments/DataSheets/MIC5332-Micropower-High-Performance-Dual-300mA-ULDO-DS20007052.pdf" (id 3) (at 106.68 26.67 0)
+      (effects (font (size 1.27 1.27)) hide)
+    )
+    (property "LCSC" "C153276" (id 4) (at 106.68 35.56 0)
       (effects (font (size 1.27 1.27)) hide)
     )
@@
     )
     (path "/65a95da7-4f7f-4162-9b7a-05aaa141d8aa"
-      (reference "Q1") (unit 1) (value "BC847BS") (footprint "Package_TO_SOT_SMD:SOT-363_SC-70-6")
+      (reference "Q1") (unit 1) (value "MMDT3904") (footprint "Package_TO_SOT_SMD:SOT-363_SC-70-6")
     )
     (path "/215c48f5-8c83-40ce-80d6-fb61d6cb6e12"
-      (reference "Q1") (unit 2) (value "BC847BS") (footprint "Package_TO_SOT_SMD:SOT-363_SC-70-6")
+      (reference "Q1") (unit 2) (value "MMDT3904") (footprint "Package_TO_SOT_SMD:SOT-363_SC-70-6")
     )
     (path "/731ee317-d717-418e-8a38-f6754143172e"
@@
     )
     (path "/6928eae3-04b8-42b2-8f00-ec0b9aa50ceb"
-      (reference "U1") (unit 1) (value "MIC5330-SSYML") (footprint "AIOC:Micrel_MLF-8-1EP_2x2mm_P0.5mm_EP0.6x1.2mm")
+      (reference "U1") (unit 1) (value "MIC5332-SSYMT") (footprint "AIOC:Micrel_MLF-8-1EP_2x2mm_P0.5mm_EP0.6x1.2mm")
     )
     (path "/374c61ba-2500-40c8-8fa4-5bb019a70699"
